Commit message: Lab 3 Done

File: src/my_r2d2/urdf/r2d2.urdf.xacro (robot description, xacro)
@@ -234,3 +234,10 @@
     <origin xyz="0.02 0 0"/>
   </joint>
+  <link name="base_footprint">
+  </link>
+  <joint name="tobaselink" type="fixed">
+    <parent link="base_footprint"/>
+    <child link="base_link"/>
+    <origin xyz="0 0 ${baselen+wheeldiam}"/>
+  </joint>
 </robot>

Commit message: Lab 4 Done

File: src/my_r2d2/urdf/r2d2.urdf.xacro (robot description, xacro)
@@ -241,3 +241,10 @@
     <origin xyz="0 0 ${baselen+wheeldiam}"/>
   </joint>
+  <link name="eye">
+  </link>
+  <joint name="toeye" type="fixed">
+    <parent link="lens"/>
+    <child link="eye"/>
+    <origin xyz="0.02 0 0"/>
+  </joint>
 </robot>

Commit message: Lab 5 Done

File: src/my_r2d2/urdf/r2d2.urdf.xacro (robot description, xacro)
@@ -246,5 +246,5 @@
     <parent link="lens"/>
     <child link="eye"/>
-    <origin xyz="0.02 0 0"/>
+    <origin rpy="0 0 -${pi/2}" xyz="0 ${pi/2} 0"/>
   </joint>
 </robot>
